File: KiCAD/Keyboard/frameortho.kicad_pcb (KiCad board)
At the start: 2 copper layers, 276 x 105 mm, 103 parts, among them J1 USB_C_Receptacle_USB2.0_16P, SW1 SW_Push, SW2 SW_Push, U1 RP2040, U2 W25Q128JVS, U3 XC6206PxxxMR, Y1 12 MHz 20pF

Commit message: mostly finished pcb
Parts:
- removed J1: USB_C_Receptacle_USB2.0_16P, ScottoKeebs_Components:USB_C_HRO_TYPE-C-31-M-14
- removed R1, R2: 5.1kΩ, Resistor_SMD:R_0402_1005Metric
- added TP1: TestPoint, TestPoint:TestPoint_Pad_D2.0mm, F.Cu at (206.8, 132.1)
- added TP10: TestPoint, TestPoint:TestPoint_Pad_D2.0mm, F.Cu at (210.8, 146.6)
- added TP11: TestPoint, TestPoint:TestPoint_Pad_D2.0mm, F.Cu at (214.7, 146.6)
- added TP12: TestPoint, TestPoint:TestPoint_Pad_D2.0mm, F.Cu at (218.6, 146.6)
- added TP13: TestPoint, TestPoint:TestPoint_Pad_D2.0mm, F.Cu at (210.8, 153.8)
- added TP14: TestPoint, TestPoint:TestPoint_Pad_D2.0mm, F.Cu at (214.7, 153.8)
- added TP15: TestPoint, TestPoint:TestPoint_Pad_D2.0mm, F.Cu at (218.6, 153.8)
- added TP16: TestPoint, TestPoint:TestPoint_Pad_D2.0mm, F.Cu at (222.5, 153.8)
- added TP17: TestPoint, TestPoint:TestPoint_Pad_D2.0mm, B.Cu at (206.2, 83.2)
- added TP18: TestPoint, TestPoint:TestPoint_Pad_D2.0mm, B.Cu at (210.2, 83.2)
- added TP19: TestPoint, TestPoint:TestPoint_Pad_D2.0mm, B.Cu at (214.3, 83.2)
- added TP2: TestPoint, TestPoint:TestPoint_Pad_D2.0mm, F.Cu at (210.8, 132.1)
- added TP20: TestPoint, TestPoint:TestPoint_Pad_D2.0mm, B.Cu at (218.3, 83.2)
- added TP21: TestPoint, TestPoint:TestPoint_Pad_D2.0mm, F.Cu at (227.7, 135.2)
- added TP22: TestPoint, TestPoint:TestPoint_Pad_D2.0mm, F.Cu at (231.7, 135.2)
- added TP3: TestPoint, TestPoint:TestPoint_Pad_D2.0mm, F.Cu at (214.7, 132.1)
- added TP4: TestPoint, TestPoint:TestPoint_Pad_D2.0mm, F.Cu at (218.6, 132.1)
- added TP5: TestPoint, TestPoint:TestPoint_Pad_D2.0mm, F.Cu at (210.8, 139.4)
- added TP6: TestPoint, TestPoint:TestPoint_Pad_D2.0mm, F.Cu at (214.7, 139.4)
- added TP7: TestPoint, TestPoint:TestPoint_Pad_D2.0mm, F.Cu at (218.6, 139.4)
- added TP8: TestPoint, TestPoint:TestPoint_Pad_D2.0mm, F.Cu at (222.5, 139.4)
- added TP9: TestPoint, TestPoint:TestPoint_Pad_D2.0mm, F.Cu at (206.8, 146.6)
- S1, S10, S11, S12, S13, S14, S15, S16, S17, S18, S19, S2, S20, S21, S22, S23, S24, S25, S26, S27, S28, S29, S3, S30, S31, S32, S33, S34, S35, S36, S4, S5, S6, S7, S8, S9: footprint footprint-and-cad:CPG1316S01D02_castelated_mikecinq -> Custom:CPG1316S01D02_castelated_mikecinq
Connections:
- U1 pad 11: unconnected-(U1-GPIO8-Pad11) -> GPIO8
- U1 pad 12: unconnected-(U1-GPIO9-Pad12) -> GPIO9
- U1 pad 13: unconnected-(U1-GPIO10-Pad13) -> GPIO10
- U1 pad 14: unconnected-(U1-GPIO11-Pad14) -> GPIO11
- U1 pad 15: unconnected-(U1-GPIO12-Pad15) -> GPIO12
- U1 pad 16: unconnected-(U1-GPIO13-Pad16) -> GPIO13
- U1 pad 17: unconnected-(U1-GPIO14-Pad17) -> GPIO14
- U1 pad 18: unconnected-(U1-GPIO15-Pad18) -> GPIO15
- U1 pad 2: unconnected-(U1-GPIO0-Pad2) -> COL_0
- U1 pad 27: unconnected-(U1-GPIO16-Pad27) -> COL_9
- U1 pad 28: unconnected-(U1-GPIO17-Pad28) -> COL_8
- U1 pad 29: unconnected-(U1-GPIO18-Pad29) -> COL_7
- U1 pad 3: unconnected-(U1-GPIO1-Pad3) -> COL_1
- U1 pad 30: unconnected-(U1-GPIO19-Pad30) -> COL_6
- U1 pad 31: unconnected-(U1-GPIO20-Pad31) -> COL_5
- U1 pad 32: unconnected-(U1-GPIO21-Pad32) -> GPIO21
- U1 pad 34: unconnected-(U1-GPIO22-Pad34) -> GPIO22
- U1 pad 35: unconnected-(U1-GPIO23-Pad35) -> GPIO23
- U1 pad 36: unconnected-(U1-GPIO24-Pad36) -> GPIO24
- U1 pad 37: unconnected-(U1-GPIO25-Pad37) -> GPIO25
- U1 pad 38: unconnected-(U1-GPIO26_ADC0-Pad38) -> ROW_3
- U1 pad 39: unconnected-(U1-GPIO27_ADC1-Pad39) -> ROW_2
- U1 pad 4: unconnected-(U1-GPIO2-Pad4) -> COL_2
- U1 pad 40: unconnected-(U1-GPIO28_ADC2-Pad40) -> ROW_1
- U1 pad 41: unconnected-(U1-GPIO29_ADC3-Pad41) -> ROW_0
- U1 pad 5: unconnected-(U1-GPIO3-Pad5) -> COL_3
- U1 pad 6: unconnected-(U1-GPIO4-Pad6) -> COL_4
- U1 pad 7: unconnected-(U1-GPIO5-Pad7) -> GPIO5
- U1 pad 8: unconnected-(U1-GPIO6-Pad8) -> GPIO6
- U1 pad 9: unconnected-(U1-GPIO7-Pad9) -> GPIO7
Routing:
- net ROW_2: track 0.00 -> 298.1 mm, vias 0 -> 2
- net ROW_1: track 0.00 -> 262.6 mm, vias 0 -> 2
- net ROW_0: track 0.00 -> 234.2 mm, vias 0 -> 2
- net ROW_3: track 0.00 -> 211.8 mm
- net COL_0: track 0.00 -> 162.5 mm, vias 0 -> 1
- net COL_2: track 0.37 -> 151.7 mm, vias 0 -> 1
- net COL_7: track 0.00 -> 145.0 mm, vias 0 -> 3
- net COL_6: track 0.00 -> 133.9 mm, vias 0 -> 3
- net COL_9: track 0.00 -> 133.7 mm, vias 0 -> 1
- net COL_1: track 0.00 -> 133.0 mm, vias 0 -> 1
- net COL_3: track 0.00 -> 126.7 mm, vias 0 -> 1
- net COL_8: track 0.00 -> 114.7 mm, vias 0 -> 3
- net COL_5: track 0.00 -> 113.2 mm, vias 0 -> 3
- net COL_4: track 0.00 -> 110.7 mm, vias 0 -> 1
- net GPIO13: track 0.00 -> 65.1 mm
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Other:
- board text added: "5V"
- board text added: "Boot"
- board text added: "D+"
- board text added: "D-"
- board text added: "GND"
- board text added: "GPIO10"
- board text added: "GPIO11"
- board text added: "GPIO12"
- board text added: "GPIO13"
- board text added: "GPIO14"
- board text added: "GPIO15"
- board text added: "GPIO16"
- board text added: "GPIO22"
- board text added: "GPIO23"
- board text added: "GPIO24"
- board text added: "GPIO25"
- board text added: "GPIO5"
- board text added: "GPIO6"
- board text added: "GPIO7"
- board text added: "GPIO8"
- board text added: "GPIO9"
- board text added: "Reset"
- board text added: "SWCLK"
- board text added: "SWDIO"
