File: KiCAD/Keyboard/matrix.kicad_sch (KiCad schematic)
At the start: 0 parts

Commit message: start keyboard pcb
Parts:
- added D1, D10, D11, D12, D13, D14, D15, D16, D17, D18, D19, D2, D20, D21, D22, D23, D24, D25, D26, D27, D28, D29, D3, D30, D31, D32, D33, D34, D35, D36, D4, D5, D6, D7, D8, D9: D_Small, ScottoKeebs_Components:Diode_SOD-123, symbol Device:D_Small
- added S1, S10, S11, S12, S13, S14, S15, S16, S17, S18, S19, S2, S20, S21, S22, S23, S24, S25, S26, S27, S28, S29, S3, S30, S31, S32, S33, S34, S35, S36, S4, S5, S6, S7, S8, S9: Keyswitch, footprint-and-cad:CPG1316S01D02_castelated_mikecinq, symbol Custom:Placeholder_Keyswitch_GND
Connections:
- new net: D12.2 (A), S12.2
- new net: D30.2 (A), S30.2
- new net: D19.2 (A), S19.2
- new net: D13.2 (A), S13.2
- new net: D24.2 (A), S24.2
- new net: D10.2 (A), S10.2
- new net: D36.2 (A), S36.2
- new net: D23.2 (A), S23.2
- new net: D18.2 (A), S18.2
- new net: D33.2 (A), S33.2
- new net: D7.2 (A), S7.2
- new net: D22.2 (A), S22.2
- new net: D4.2 (A), S4.2
- new net: D34.2 (A), S34.2
- new net: D2.2 (A), S2.2
- new net: D15.2 (A), S15.2
- new net: D5.2 (A), S5.2
- new net: D8.2 (A), S8.2
- new net: D6.2 (A), S6.2
- new net: D17.2 (A), S17.2
- new net: D29.2 (A), S29.2
- new net: D31.2 (A), S31.2
- new net: D16.2 (A), S16.2
- new net: D14.2 (A), S14.2
- new net: D20.2 (A), S20.2
- new net: D26.2 (A), S26.2
- new net: D21.2 (A), S21.2
- new net: D11.2 (A), S11.2
- new net: D1.2 (A), S1.2
- new net: D9.2 (A), S9.2
- new net: D32.2 (A), S32.2
- new net: D35.2 (A), S35.2
- new net: D3.2 (A), S3.2
- new net: D28.2 (A), S28.2
- new net: D27.2 (A), S27.2
- new net: D25.2 (A), S25.2
- new net COL_0: S1.1, S11.1, S21.1
- new net COL_1: S12.1, S2.1, S22.1
- new net COL_2: S13.1, S23.1, S3.1, S31.1
- new net COL_3: S14.1, S24.1, S32.1, S4.1
- new net COL_4: S15.1, S25.1, S33.1, S5.1
- new net COL_5: S16.1, S26.1, S34.1, S6.1
- new net COL_6: S17.1, S27.1, S35.1, S7.1
- new net COL_7: S18.1, S28.1, S36.1, S8.1
- new net COL_8: S19.1, S29.1, S9.1
- new net COL_9: S10.1, S20.1, S30.1
- new net GND: S1.3, S10.3, S11.3, S12.3, S13.3, S14.3, S15.3, S16.3, S17.3, S18.3, S19.3, S2.3, S20.3, S21.3, S22.3, S23.3, S24.3, S25.3, S26.3, S27.3, S28.3, S29.3, S3.3, S30.3, S31.3, S32.3, S33.3, S34.3, S35.3, S36.3, S4.3, S5.3, S6.3, S7.3, S8.3, S9.3
- new net ROW_0: D1.1 (K), D10.1 (K), D2.1 (K), D3.1 (K), D4.1 (K), D5.1 (K), D6.1 (K), D7.1 (K), D8.1 (K), D9.1 (K)
- new net ROW_1: D11.1 (K), D12.1 (K), D13.1 (K), D14.1 (K), D15.1 (K), D16.1 (K), D17.1 (K), D18.1 (K), D19.1 (K), D20.1 (K)
- new net ROW_2: D21.1 (K), D22.1 (K), D23.1 (K), D24.1 (K), D25.1 (K), D26.1 (K), D27.1 (K), D28.1 (K), D29.1 (K), D30.1 (K)
- new net ROW_3: D31.1 (K), D32.1 (K), D33.1 (K), D34.1 (K), D35.1 (K), D36.1 (K)

Commit message: mostly finished pcb
Parts:
- S1, S10, S11, S12, S13, S14, S15, S16, S17, S18, S19, S2, S20, S21, S22, S23, S24, S25, S26, S27, S28, S29, S3, S30, S31, S32, S33, S34, S35, S36, S4, S5, S6, S7, S8, S9: footprint footprint-and-cad:CPG1316S01D02_castelated_mikecinq -> Custom:CPG1316S01D02_castelated_mikecinq
Changed lines of the file:
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@@
 			)
 		)
-		(property "Footprint" "footprint-and-cad:CPG1316S01D02_castelated_mikecinq"
+		(property "Footprint" "Custom:CPG1316S01D02_castelated_mikecinq"
 			(at 91.44 97.79 0)
 			(effects
@@
 			)
 		)
-		(property "Footprint" "footprint-and-cad:CPG1316S01D02_castelated_mikecinq"
+		(property "Footprint" "Custom:CPG1316S01D02_castelated_mikecinq"
 			(at 205.74 116.84 0)
 			(effects
@@
 			)
 		)
-		(property "Footprint" "footprint-and-cad:CPG1316S01D02_castelated_mikecinq"
+		(property "Footprint" "Custom:CPG1316S01D02_castelated_mikecinq"
 			(at 193.04 97.79 0)
 			(effects
@@
 			)
 		)
-		(property "Footprint" "footprint-and-cad:CPG1316S01D02_castelated_mikecinq"
+		(property "Footprint" "Custom:CPG1316S01D02_castelated_mikecinq"
 			(at 116.84 116.84 0)
 			(effects
@@
 			)
 		)
-		(property "Footprint" "footprint-and-cad:CPG1316S01D02_castelated_mikecinq"
+		(property "Footprint" "Custom:CPG1316S01D02_castelated_mikecinq"
 			(at 205.74 78.74 0)
 			(effects
@@
 			)
 		)
-		(property "Footprint" "footprint-and-cad:CPG1316S01D02_castelated_mikecinq"
+		(property "Footprint" "Custom:CPG1316S01D02_castelated_mikecinq"
 			(at 180.34 135.89 0)
 			(effects
@@
 			)
 		)
-		(property "Footprint" "footprint-and-cad:CPG1316S01D02_castelated_mikecinq"
+		(property "Footprint" "Custom:CPG1316S01D02_castelated_mikecinq"
 			(at 104.14 116.84 0)
 			(effects
@@
 			)
 		)
-		(property "Footprint" "footprint-and-cad:CPG1316S01D02_castelated_mikecinq"
+		(property "Footprint" "Custom:CPG1316S01D02_castelated_mikecinq"
 			(at 91.44 116.84 0)
 			(effects
@@
 			)
 		)
-		(property "Footprint" "footprint-and-cad:CPG1316S01D02_castelated_mikecinq"
+		(property "Footprint" "Custom:CPG1316S01D02_castelated_mikecinq"
 			(at 91.44 78.74 0)
 			(effects
@@
 			)
 		)
-		(property "Footprint" "footprint-and-cad:CPG1316S01D02_castelated_mikecinq"
+		(property "Footprint" "Custom:CPG1316S01D02_castelated_mikecinq"
 			(at 129.54 78.74 0)
 			(effects
@@
 			)
 		)
-		(property "Footprint" "footprint-and-cad:CPG1316S01D02_castelated_mikecinq"
+		(property "Footprint" "Custom:CPG1316S01D02_castelated_mikecinq"
 			(at 180.34 78.74 0)
 			(effects
@@
 			)
 		)
-		(property "Footprint" "footprint-and-cad:CPG1316S01D02_castelated_mikecinq"
+		(property "Footprint" "Custom:CPG1316S01D02_castelated_mikecinq"
 			(at 154.94 135.89 0)
 			(effects
@@
 			)
 		)
-		(property "Footprint" "footprint-and-cad:CPG1316S01D02_castelated_mikecinq"
+		(property "Footprint" "Custom:CPG1316S01D02_castelated_mikecinq"
 			(at 180.34 97.79 0)
 			(effects
@@
 			)
 		)
-		(property "Footprint" "footprint-and-cad:CPG1316S01D02_castelated_mikecinq"
+		(property "Footprint" "Custom:CPG1316S01D02_castelated_mikecinq"
 			(at 167.64 97.79 0)
 			(effects
@@
 			)
 		)
-		(property "Footprint" "footprint-and-cad:CPG1316S01D02_castelated_mikecinq"
+		(property "Footprint" "Custom:CPG1316S01D02_castelated_mikecinq"
 			(at 193.04 116.84 0)
 			(effects
@@
 			)
 		)
-		(property "Footprint" "footprint-and-cad:CPG1316S01D02_castelated_mikecinq"
+		(property "Footprint" "Custom:CPG1316S01D02_castelated_mikecinq"
 			(at 104.14 135.89 0)
 			(effects
@@
 			)
 		)
-		(property "Footprint" "footprint-and-cad:CPG1316S01D02_castelated_mikecinq"
+		(property "Footprint" "Custom:CPG1316S01D02_castelated_mikecinq"
 			(at 154.94 78.74 0)
 			(effects
@@
 			)
 		)
-		(property "Footprint" "footprint-and-cad:CPG1316S01D02_castelated_mikecinq"
+		(property "Footprint" "Custom:CPG1316S01D02_castelated_mikecinq"
 			(at 116.84 78.74 0)
 			(effects
@@
 			)
 		)
-		(property "Footprint" "footprint-and-cad:CPG1316S01D02_castelated_mikecinq"
+		(property "Footprint" "Custom:CPG1316S01D02_castelated_mikecinq"
 			(at 78.74 116.84 0)
 			(effects
@@
 			)
 		)
-		(property "Footprint" "footprint-and-cad:CPG1316S01D02_castelated_mikecinq"
+		(property "Footprint" "Custom:CPG1316S01D02_castelated_mikecinq"
 			(at 78.74 97.79 0)
 			(effects
@@
 			)
 		)
-		(property "Footprint" "footprint-and-cad:CPG1316S01D02_castelated_mikecinq"
+		(property "Footprint" "Custom:CPG1316S01D02_castelated_mikecinq"
 			(at 193.04 78.74 0)
 			(effects
@@
 			)
 		)
-		(property "Footprint" "footprint-and-cad:CPG1316S01D02_castelated_mikecinq"
+		(property "Footprint" "Custom:CPG1316S01D02_castelated_mikecinq"
 			(at 116.84 135.89 0)
 			(effects
@@
 			)
 		)
-		(property "Footprint" "footprint-and-cad:CPG1316S01D02_castelated_mikecinq"
+		(property "Footprint" "Custom:CPG1316S01D02_castelated_mikecinq"
 			(at 167.64 135.89 0)
 			(effects
@@
 			)
 		)
-		(property "Footprint" "footprint-and-cad:CPG1316S01D02_castelated_mikecinq"
+		(property "Footprint" "Custom:CPG1316S01D02_castelated_mikecinq"
 			(at 116.84 97.79 0)
 			(effects
@@
 			)
 		)
-		(property "Footprint" "footprint-and-cad:CPG1316S01D02_castelated_mikecinq"
+		(property "Footprint" "Custom:CPG1316S01D02_castelated_mikecinq"
 			(at 154.94 97.79 0)
 			(effects
@@
 			)
 		)
-		(property "Footprint" "footprint-and-cad:CPG1316S01D02_castelated_mikecinq"
+		(property "Footprint" "Custom:CPG1316S01D02_castelated_mikecinq"
 			(at 180.34 116.84 0)
 			(effects
@@
 			)
 		)
-		(property "Footprint" "footprint-and-cad:CPG1316S01D02_castelated_mikecinq"
+		(property "Footprint" "Custom:CPG1316S01D02_castelated_mikecinq"
 			(at 154.94 116.84 0)
 			(effects
@@
 			)
 		)
-		(property "Footprint" "footprint-and-cad:CPG1316S01D02_castelated_mikecinq"
+		(property "Footprint" "Custom:CPG1316S01D02_castelated_mikecinq"
 			(at 167.64 116.84 0)
 			(effects
@@
 			)
 		)
-		(property "Footprint" "footprint-and-cad:CPG1316S01D02_castelated_mikecinq"
+		(property "Footprint" "Custom:CPG1316S01D02_castelated_mikecinq"
 			(at 205.74 97.79 0)
 			(effects
@@
 			)
 		)
-		(property "Footprint" "footprint-and-cad:CPG1316S01D02_castelated_mikecinq"
+		(property "Footprint" "Custom:CPG1316S01D02_castelated_mikecinq"
 			(at 129.54 97.79 0)
 			(effects
@@
 			)
 		)
-		(property "Footprint" "footprint-and-cad:CPG1316S01D02_castelated_mikecinq"
+		(property "Footprint" "Custom:CPG1316S01D02_castelated_mikecinq"
 			(at 78.74 78.74 0)
 			(effects
@@
 			)
 		)
-		(property "Footprint" "footprint-and-cad:CPG1316S01D02_castelated_mikecinq"
+		(property "Footprint" "Custom:CPG1316S01D02_castelated_mikecinq"
 			(at 129.54 116.84 0)
 			(effects
@@
 			)
 		)
-		(property "Footprint" "footprint-and-cad:CPG1316S01D02_castelated_mikecinq"
+		(property "Footprint" "Custom:CPG1316S01D02_castelated_mikecinq"
 			(at 167.64 78.74 0)
 			(effects
@@
 			)
 		)
-		(property "Footprint" "footprint-and-cad:CPG1316S01D02_castelated_mikecinq"
+		(property "Footprint" "Custom:CPG1316S01D02_castelated_mikecinq"
 			(at 129.54 135.89 0)
 			(effects
@@
 			)
 		)
-		(property "Footprint" "footprint-and-cad:CPG1316S01D02_castelated_mikecinq"
+		(property "Footprint" "Custom:CPG1316S01D02_castelated_mikecinq"
 			(at 104.14 97.79 0)
 			(effects
@@
 			)
 		)
-		(property "Footprint" "footprint-and-cad:CPG1316S01D02_castelated_mikecinq"
+		(property "Footprint" "Custom:CPG1316S01D02_castelated_mikecinq"
 			(at 104.14 78.74 0)
 			(effects
