File: KiCAD/USB/usb-hub.kicad_sch (KiCad schematic)
At the start: 22 parts, among them J1 046809610110846+ Male, J2 046809610110846+ Female, J3 Conn_01x04_Socket, U1 CY7C65634-28LTXC, Y1 12MHz 20pF

Commit message: start keyboard pcb
Parts:
- C10, C9: value 30 pF -> 33 pF
Changed lines of the file:
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@@
 			)
 		)
-		(property "Value" "30 pF"
+		(property "Value" "33 pF"
 			(at 81.2863 134.62 0)
 			(effects
@@
 			)
 		)
-		(property "Value" "30 pF"
+		(property "Value" "33 pF"
 			(at 104.394 134.62 0)
 			(effects

Commit message: why no commit
Parts:
- Y1: value 12MHz 20pF -> 12MHz 18pF
Other:
- note added: "C(L)=2*(C(Xtal)-C(Stray))=2*(18-5)=26pF->27pF"
- note removed: "C(L)=2*(C(Xtal)-C(Stray))=2*(20-4)=32pF->33pF"
Changed lines of the file:
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@@
 		)
 	)
-	(text "C(L)=2*(C(Xtal)-C(Stray))=2*(20-4)=32pF->33pF"
+	(text "C(L)=2*(C(Xtal)-C(Stray))=2*(18-5)=26pF->27pF"
 		(exclude_from_sim no)
 		(at 91.694 151.384 0)
@@
 			)
 		)
-		(property "Value" "12MHz 20pF"
+		(property "Value" "12MHz 18pF"
 			(at 92.71 123.952 0)
 			(effects
