File: KiCAD/Display Adapters/Display Adapters.kicad_sch (KiCad schematic)
At the start: 1 part, among them J1 20455-040E-76

Commit message: most of the edp to dp
Parts:
- added J2: G46M2023201BTWEU, G46M2023201BTWEU:AMPHENOL_G46M2023201BTWEU, symbol G46M2023201BTWEU:G46M2023201BTWEU
- added J3: XT30PW-M, XT30PW-M:AMASS_XT30PW-M, symbol XT30PW-M:XT30PW-M
Connections:
- net GNDD: now also J1.24, J1.25, J1.26
- net 1_EDP_TX_P: now reaches J1.10
- net 1_EDP_TX_P: now also J2.9 (ML_LANE1_P)
- net 0_EDP_TX_N: now reaches J1.12
- net 0_EDP_TX_N: now also J2.5 (ML_LANE0_N)
- net 0_EDP_TX_P: now reaches J1.13
- net 0_EDP_TX_P: now also J2.3 (ML_LANE0_P)
- net AUX_P: now reaches J1.15
- net AUX_P: now also J2.16 (AUX_CH_P)
- net AUX_N: now reaches J1.16
- net AUX_N: now also J2.18 (AUX_CH_N)
- net +3.3V: now reaches J1.18
- net +3.3V: now also J1.19, J1.20, J1.21, J2.20 (DP_PWR)
- net SELF_TEST: now reaches J1.22
- net EDP_HPD: now reaches J1.27
- net EDP_HPD: now also J2.2 (HOTPLUG_DETECT)
- net GND: now reaches J1.28
- net GND: now also J1.29, J1.30, J1.31
- net 3_EDP_TX_N: now reaches J1.3
- net 3_EDP_TX_N: now also J2.12 (ML_LANE3_N)
- net BLK_OFF_N: now reaches J1.32
- net BLK_PWM_LCD: now reaches J1.33
- net +5V: now reaches J1.36
- net +5V: now also J1.37, J1.38, J1.39, J3.P
- net 3_EDP_TX_P: now reaches J1.4
- net 3_EDP_TX_P: now also J2.10 (ML_LANE3_P)
- net 2_EDP_TX_N: now reaches J1.6
- net 2_EDP_TX_N: now also J2.17 (ML_LANE2_N)
- net 2_EDP_TX_P: now reaches J1.7
- net 2_EDP_TX_P: now also J2.15 (ML_LANE2_P)
- net 1_EDP_TX_N: now reaches J1.9
- net 1_EDP_TX_N: now also J2.11 (ML_LANE1_N)
- net GNDREF: now reaches J1.S1 (SHIELD), J1.S2 (SHIELD), J1.S3 (SHIELD), J1.S4 (SHIELD)
- net GNDREF: now also J2.SH1 (SHIELD), J2.SH2 (SHIELD), J2.SH3 (SHIELD), J2.SH4 (SHIELD), J3.N
